Commit message: Changes omav.xacro

File: rotors_description/urdf/omav.xacro (robot description, xacro)
@@ -80,6 +80,6 @@
   <xacro:double_tilt_unit robot_namespace="${namespace}"
     suffix="right"
-    direction_upper="cw"
-    direction_lower="cw"
+    direction_upper="ccw"
+    direction_lower="ccw"
     motor_constant="${motor_constant}"
     motor_constant_lower="${motor_constant_lower}"
@@ -105,6 +105,6 @@
     robot_namespace="${namespace}"
     suffix="left"
-    direction_upper="ccw"
-    direction_lower="ccw"
+    direction_upper="cw"
+    direction_lower="cw"
     motor_constant="${motor_constant}"
     motor_constant_lower="${motor_constant_lower}"
@@ -130,4 +130,28 @@
     robot_namespace="${namespace}"
     suffix="front_left"
+    direction_upper="ccw"
+    direction_lower="ccw"
+    motor_constant="${motor_constant}"
+    motor_constant_lower="${motor_constant_lower}"
+    moment_constant="${moment_constant}"
+    moment_constant_lower="${moment_constant_lower}"
+    parent="${namespace}/base_link"
+    mass_rotor="${mass_rotor}"
+    mass_tilt_unit="${mass_tilt_unit}"
+    time_constant_up="${time_constant_up}"
+    time_constant_down="${time_constant_down}"
+    max_rot_velocity="${max_rot_velocity}"
+    rotor_offset_top="${rotor_offset_top}"
+    motor_number="2"
+    rotor_drag_coefficient="${rotor_drag_coefficient}"
+    rolling_moment_coefficient="${rolling_moment_coefficient}"
+    mesh="propeller"
+    mesh_tilt_unit="${mesh_file_tilt_unit}"
+    color="Orange">
+    <origin xyz="${cos30*arm_length} ${sin30*arm_length} 0" rpy="0 0 0.52359877559"/>
+    <xacro:insert_block name="rotor_inertia" />
+  </xacro:double_tilt_unit>
+  <xacro:double_tilt_unit robot_namespace="${namespace}"
+    suffix="back_right"
     direction_upper="cw"
     direction_lower="cw"
@@ -143,5 +167,29 @@
     max_rot_velocity="${max_rot_velocity}"
     rotor_offset_top="${rotor_offset_top}"
-    motor_number="2"
+    motor_number="3"
+    rotor_drag_coefficient="${rotor_drag_coefficient}"
+    rolling_moment_coefficient="${rolling_moment_coefficient}"
+    mesh="propeller"
+    mesh_tilt_unit="${mesh_file_tilt_unit}"
+    color="DarkGrey">
+    <origin xyz="-${cos30*arm_length} -${sin30*arm_length} 0" rpy="0 0 3.66519142919"/>
+    <xacro:insert_block name="rotor_inertia" />
+  </xacro:double_tilt_unit>
+  <xacro:double_tilt_unit robot_namespace="${namespace}"
+    suffix="front_right"
+    direction_upper="cw"
+    direction_lower="cw"
+    motor_constant="${motor_constant}"
+    motor_constant_lower="${motor_constant_lower}"
+    moment_constant="${moment_constant}"
+    moment_constant_lower="${moment_constant_lower}"
+    parent="${namespace}/base_link"
+    mass_rotor="${mass_rotor}"
+    mass_tilt_unit="${mass_tilt_unit}"
+    time_constant_up="${time_constant_up}"
+    time_constant_down="${time_constant_down}"
+    max_rot_velocity="${max_rot_velocity}"
+    rotor_offset_top="${rotor_offset_top}"
+    motor_number="4"
     rotor_drag_coefficient="${rotor_drag_coefficient}"
     rolling_moment_coefficient="${rolling_moment_coefficient}"
@@ -149,59 +197,11 @@
     mesh_tilt_unit="${mesh_file_tilt_unit}"
     color="Orange">
-    <origin xyz="${cos30*arm_length} ${sin30*arm_length} 0" rpy="0 0 0.52359877559"/>
+    <origin xyz="${cos30*arm_length} -${sin30*arm_length} 0" rpy="0 0 5.75958653158"/>
     <xacro:insert_block name="rotor_inertia" />
   </xacro:double_tilt_unit>
   <xacro:double_tilt_unit robot_namespace="${namespace}"
-    suffix="back_right"
+    suffix="back_left"
     direction_upper="ccw"
     direction_lower="ccw"
-    motor_constant="${motor_constant}"
-    motor_constant_lower="${motor_constant_lower}"
-    moment_constant="${moment_constant}"
-    moment_constant_lower="${moment_constant_lower}"
-    parent="${namespace}/base_link"
-    mass_rotor="${mass_rotor}"
-    mass_tilt_unit="${mass_tilt_unit}"
-    time_constant_up="${time_constant_up}"
-    time_constant_down="${time_constant_down}"
-    max_rot_velocity="${max_rot_velocity}"
-    rotor_offset_top="${rotor_offset_top}"
-    motor_number="3"
-    rotor_drag_coefficient="${rotor_drag_coefficient}"
-    rolling_moment_coefficient="${rolling_moment_coefficient}"
-    mesh="propeller"
-    mesh_tilt_unit="${mesh_file_tilt_unit}"
-    color="DarkGrey">
-    <origin xyz="-${cos30*arm_length} -${sin30*arm_length} 0" rpy="0 0 3.66519142919"/>
-    <xacro:insert_block name="rotor_inertia" />
-  </xacro:double_tilt_unit>
-  <xacro:double_tilt_unit robot_namespace="${namespace}"
-    suffix="front_right"
-    direction_upper="ccw"
-    direction_lower="ccw"
-    motor_constant="${motor_constant}"
-    motor_constant_lower="${motor_constant_lower}"
-    moment_constant="${moment_constant}"
-    moment_constant_lower="${moment_constant_lower}"
-    parent="${namespace}/base_link"
-    mass_rotor="${mass_rotor}"
-    mass_tilt_unit="${mass_tilt_unit}"
-    time_constant_up="${time_constant_up}"
-    time_constant_down="${time_constant_down}"
-    max_rot_velocity="${max_rot_velocity}"
-    rotor_offset_top="${rotor_offset_top}"
-    motor_number="4"
-    rotor_drag_coefficient="${rotor_drag_coefficient}"
-    rolling_moment_coefficient="${rolling_moment_coefficient}"
-    mesh="propeller"
-    mesh_tilt_unit="${mesh_file_tilt_unit}"
-    color="Orange">
-    <origin xyz="${cos30*arm_length} -${sin30*arm_length} 0" rpy="0 0 5.75958653158"/>
-    <xacro:insert_block name="rotor_inertia" />
-  </xacro:double_tilt_unit>
-  <xacro:double_tilt_unit robot_namespace="${namespace}"
-    suffix="back_left"
-    direction_upper="cw"
-    direction_lower="cw"
     motor_constant="${motor_constant}"
     motor_constant_lower="${motor_constant_lower}"
